File: KiCAD/Pluralsight_Drumkit/Pluralsight_Drumkit.sch (KiCad schematic (older format))
At the start: 24 parts, among them J1 DIN-5_180degree, J2 Solenoid Connector, J3 Prog Jumper, J4 Power, P1 Digital, P10 CONN_01X01, P11 CONN_01X01, P12 CONN_01X01, P13 CONN_01X01, P2 Power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

Commit message: Added Digikey BOM
Parts:
- J1: value DIN-5_180degree -> MIDI DIN
Changed lines of the file:
@@
 P 1450 1325
 F 0 "J1" H 1575 1550 50  0000 C CNN
-F 1 "DIN-5_180degree" H 1450 1075 50  0000 C CNN
+F 1 "MIDI DIN" H 1450 1075 50  0000 C CNN
 F 2 "Connectors:SDS-50J" H 1450 1325 50  0001 C CNN
 F 3 "http://www.mouser.com/ds/2/18/40_c091_abd_e-75918.pdf" H 1450 1325 50  0001 C CNN
